File: Aviônica 2.0 - Para corrosão/esquema.brd (EAGLE design)
At the start: 100 x 62.2 mm, 8 parts

Commit message: Placa do paraquedas
Parts:
- removed U$7: JST2.54X2P, CRD:JST2.54X2P_FOOTPRINT
Connections:
- removed net N$7: U$2.VCC, U$4.5V
- net GND: no longer U$7.2
- net VIN: now also U$2.VCC, U$4.5V; no longer U$7.1
Routing:
- net VIN: track 14.7 -> 116.0 mm
- net N$7: track 40.0 -> 0.00 mm
Changed lines of the file:
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@@
 </layers>
 <board>
-<fusionsync huburn="a.YnVzaW5lc3M6ZGlzY2VudGU3MA" projecturn="a.YnVzaW5lc3M6ZGlzY2VudGU3MCMyMDIyMDIxNzQ5ODU5MDQ4MQ" f3durn="urn:adsk.wipprod:dm.lineage:HlMlsNpuT-m1BwDsnHgy8Q" pcbguid="" lastpulledtime="" lastsyncedchangeguid="" latestrevisionid="07065a72-c239-4b71-a72c-e7634940160a" lastsyncedrevisionid="07065a72-c239-4b71-a72c-e7634940160a" lastboardhashguid="f4d7ea46-0b2e-5c52-99f8-57296fa67e67" lastpushedtime="2023-03-13T13:09:58Z" linktopcb3d="true"/>
+<fusionsync huburn="a.YnVzaW5lc3M6ZGlzY2VudGU3MA" projecturn="a.YnVzaW5lc3M6ZGlzY2VudGU3MCMyMDIyMDIxNzQ5ODU5MDQ4MQ" f3durn="urn:adsk.wipprod:dm.lineage:HlMlsNpuT-m1BwDsnHgy8Q" pcbguid="" lastpulledtime="" lastsyncedchangeguid="" latestrevisionid="41cdf830-8c3a-4f2d-939e-ec135ec38c11" lastsyncedrevisionid="41cdf830-8c3a-4f2d-939e-ec135ec38c11" lastboardhashguid="9d6c18a2-fee8-5258-f283-1b11a8ffe41c" lastpushedtime="2023-03-13T20:35:54Z" linktopcb3d="true"/>
 <plain>
 <wire x1="0" y1="-0.08" x2="99.97" y2="0.02" width="0" layer="20"/>
@@
 <element name="U$6" library="CRD" library_urn="urn:adsk.eagle:library:39051337" package="SWITCH_3PIN" package3d_urn="urn:adsk.eagle:package:39192263/4" value="SWITCH_3PIN" x="7" y="24" smashed="yes" rot="R90"/>
 <element name="U$4" library="CRD" library_urn="urn:adsk.eagle:library:39051337" package="WIFI_KIT32" package3d_urn="urn:adsk.eagle:package:39051622/4" value="WIFI_KIT32" x="48" y="40" smashed="yes" rot="R180"/>
-<element name="U$7" library="CRD" library_urn="urn:adsk.eagle:library:39051337" package="JST2.54X2P_FOOTPRINT" package3d_urn="urn:adsk.eagle:package:39191967/2" value="JST2.54X2P" x="8.5" y="36" smashed="yes" rot="R270"/>
 <element name="JP1" library="pinhead" library_urn="urn:adsk.eagle:library:325" package="1X01" package3d_urn="urn:adsk.eagle:package:22485/2" value="" x="32" y="38" smashed="yes">
 <attribute name="NAME" x="30.6538" y="39.8288" size="1.27" layer="25" ratio="10"/>
@@
 <wire x1="80" y1="47.14894375" x2="80" y2="49" width="1" layer="1"/>
 </signal>
-<signal name="N$7">
+<signal name="GND">
+<contactref element="U$5" pad="2"/>
+<contactref element="U$1" pad="GND"/>
+<contactref element="U$3" pad="GND"/>
+<contactref element="U$2" pad="GND"/>
+<contactref element="U$4" pad="GND_1"/>
+<contactref element="U$4" pad="GND_2"/>
+<polygon width="1" layer="1">
+<vertex x="1" y="61"/>
+<vertex x="1" y="1"/>
+<vertex x="99" y="1"/>
+<vertex x="99" y="61"/>
+</polygon>
+<wire x1="8.54" y1="10.84" x2="26.97" y2="13.4255" width="0" layer="19" extent="1-1"/>
+</signal>
+<signal name="VIN">
+<contactref element="U$6" pad="3"/>
 <contactref element="U$2" pad="VCC"/>
 <contactref element="U$4" pad="5V"/>
@@
 <wire x1="62" y1="14.26" x2="62" y2="27" width="1" layer="1"/>
 <wire x1="62" y1="27" x2="65" y2="30" width="1" layer="1"/>
-</signal>
-<signal name="GND">
-<contactref element="U$5" pad="2"/>
-<contactref element="U$1" pad="GND"/>
-<contactref element="U$3" pad="GND"/>
-<contactref element="U$2" pad="GND"/>
-<contactref element="U$4" pad="GND_1"/>
-<contactref element="U$7" pad="2"/>
-<contactref element="U$4" pad="GND_2"/>
-<polygon width="1" layer="1">
-<vertex x="1" y="61"/>
-<vertex x="1" y="1"/>
-<vertex x="99" y="1"/>
-<vertex x="99" y="61"/>
-</polygon>
-<wire x1="59.77" y1="9.49" x2="70.506" y2="25.305" width="0" layer="19" extent="1-1"/>
-<wire x1="36.77" y1="9.49" x2="59.77" y2="9.49" width="0" layer="19" extent="1-1"/>
-<wire x1="26.97" y1="13.4255" x2="36.77" y2="9.49" width="0" layer="19" extent="1-1"/>
-<wire x1="8.54" y1="10.84" x2="26.97" y2="13.4255" width="0" layer="19" extent="1-1"/>
-<wire x1="27.1845" y1="35.5555" x2="26.97" y2="13.4255" width="0" layer="19" extent="1-1"/>
-<wire x1="8.5" y1="34.73" x2="27.1845" y2="35.5555" width="0" layer="19" extent="1-1"/>
-</signal>
-<signal name="VIN">
-<contactref element="U$6" pad="3"/>
-<contactref element="U$7" pad="1"/>
 <wire x1="8.6" y1="27" x2="10" y2="27" width="1" layer="1"/>
-<wire x1="12" y1="29" x2="10" y2="27" width="1" layer="1"/>
-<wire x1="8.5" y1="37.27" x2="9.73" y2="37.27" width="1" layer="1"/>
-<wire x1="9.73" y1="37.27" x2="12" y2="35" width="1" layer="1"/>
-<wire x1="12" y1="35" x2="12" y2="29" width="1" layer="1"/>
+<wire x1="10" y1="27" x2="15" y2="22" width="1" layer="1"/>
+<wire x1="15" y1="22" x2="15" y2="6" width="1" layer="1"/>
+<wire x1="15" y1="6" x2="18" y2="3" width="1" layer="1"/>
+<wire x1="25.14894375" y1="3" x2="25.16494375" y2="2.984" width="1" layer="1"/>
+<wire x1="25.16494375" y1="2.984" x2="51.984" y2="2.984" width="1" layer="1"/>
+<wire x1="51.984" y1="2.984" x2="57" y2="8" width="1" layer="1"/>
+<wire x1="58.03" y1="12.03" x2="59.77" y2="12.03" width="1" layer="1"/>
+<wire x1="18" y1="3" x2="25.14894375" y2="3" width="1" layer="1"/>
+<wire x1="57" y1="8" x2="57" y2="11" width="1" layer="1"/>
+<wire x1="57" y1="11" x2="58.03" y2="12.03" width="1" layer="1"/>
 </signal>
 <signal name="N$4">
