File: Aviônica 3.0 - Para corrosão/esquema.brd (EAGLE design)
At the start: 100 x 62.2 mm, 7 parts

Commit message: Placa do paraquedas
Parts:
- added U$7: GPS_MODULE, CRD:GPS_MODULE_FOOTPRINT
- added U$8: GPS_ANTENNA, CRD:GPS_ANTENNA_FOOTPRINT
- moved JP1 55.0 mm to (84.0, 56.0)
- moved U$3 6.20 mm to (16.9, 35.7)
- moved U$1 1.62 mm to (20.8, 15.7), flipped to the bottom, turned to 270 degrees
- moved U$2 0.97 mm to (84.2, 18.0), flipped to the bottom, turned to 90 degrees
Routing:
- net MOSI: track 124.3 -> 78.0 mm
- net N$2: track 12.6 -> 51.6 mm
- net N$1: track 70.0 -> 32.0 mm
- net SCLK: track 57.0 -> 25.7 mm
- net VIN: track 116.0 -> 86.6 mm
- net SCL: track 100.8 -> 85.9 mm
- net MISO: track 35.5 -> 23.1 mm
- net N$4: track 36.9 -> 30.2 mm
- net SDA: track 48.5 -> 54.1 mm
