File: Aviônica 3.0 - Para corrosão/esquema.sch (EAGLE design)
At the start: 8 parts

Commit message: Placa do paraquedas
Parts:
- added U$8: GPS_ANTENNA, CRD:GPS_ANTENNA
- U$7: value JST2.54X2P -> GPS_MODULE; device CRD:JST2.54X2P -> CRD:GPS_MODULE
Connections:
- removed net N$7: U$2.VCC, U$4.5V
- net GND: no longer U$7.2
- net VIN: now also U$2.VCC, U$4.5V; no longer U$7.1
Changed lines of the file:
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@@
 <part name="GND3" library="supply1" library_urn="urn:adsk.eagle:library:371" deviceset="GND" device=""/>
 <part name="GND5" library="supply1" library_urn="urn:adsk.eagle:library:371" deviceset="GND" device=""/>
-<part name="U$7" library="CRD" library_urn="urn:adsk.eagle:library:39051337" deviceset="JST2.54X2P" device="" package3d_urn="urn:adsk.eagle:package:39191967/2"/>
-<part name="GND6" library="supply1" library_urn="urn:adsk.eagle:library:371" deviceset="GND" device=""/>
 <part name="GND7" library="supply1" library_urn="urn:adsk.eagle:library:371" deviceset="GND" device=""/>
 <part name="JP1" library="pinhead" library_urn="urn:adsk.eagle:library:325" deviceset="PINHD-1X1" device="" package3d_urn="urn:adsk.eagle:package:22485/2"/>
+<part name="U$7" library="CRD" library_urn="urn:adsk.eagle:library:39051337" deviceset="GPS_MODULE" device="" package3d_urn="urn:adsk.eagle:package:39608400/2"/>
+<part name="U$8" library="CRD" library_urn="urn:adsk.eagle:library:39051337" deviceset="GPS_ANTENNA" device="" package3d_urn="urn:adsk.eagle:package:39608528/1"/>
 </parts>
 <sheets>
@@
 <attribute name="VALUE" x="-5.08" y="55.88" size="1.778" layer="96"/>
 </instance>
-<instance part="U$7" gate="G$1" x="121.92" y="-15.24" smashed="yes"/>
-<instance part="GND6" gate="1" x="124.46" y="-33.02" smashed="yes">
-<attribute name="VALUE" x="121.92" y="-35.56" size="1.778" layer="96"/>
-</instance>
 <instance part="GND7" gate="1" x="76.2" y="48.26" smashed="yes">
 <attribute name="VALUE" x="73.66" y="45.72" size="1.778" layer="96"/>
@@
 <attribute name="VALUE" x="62.23" y="-33.02" size="1.778" layer="96"/>
 </instance>
+<instance part="U$7" gate="G$1" x="144.78" y="33.02" smashed="yes"/>
+<instance part="U$8" gate="G$1" x="144.78" y="-10.16" smashed="yes"/>
 </instances>
 <busses>
@@
 </segment>
 </net>
-<net name="N$7" class="0">
-<segment>
-<pinref part="U$2" gate="G$1" pin="VCC"/>
-<wire x1="-55.88" y1="-27.94" x2="-55.88" y2="-45.72" width="0.1524" layer="91"/>
-<wire x1="-55.88" y1="-45.72" x2="-71.12" y2="-45.72" width="0.1524" layer="91"/>
-<wire x1="-71.12" y1="-45.72" x2="-71.12" y2="43.18" width="0.1524" layer="91"/>
-<pinref part="U$4" gate="G$1" pin="5V"/>
-<wire x1="-71.12" y1="43.18" x2="1.524" y2="43.18" width="0.1524" layer="91"/>
-</segment>
-</net>
 <net name="GND" class="0">
 <segment>
@@
 </segment>
 <segment>
-<pinref part="GND6" gate="1" pin="GND"/>
-<pinref part="U$7" gate="G$1" pin="2"/>
-<wire x1="124.46" y1="-30.48" x2="124.46" y2="-25.4" width="0.1524" layer="91"/>
-</segment>
-<segment>
 <pinref part="U$4" gate="G$1" pin="GND_2"/>
 <wire x1="54.864" y1="48.26" x2="63.5" y2="48.26" width="0.1524" layer="91"/>
@@
 </segment>
 <segment>
-<pinref part="U$7" gate="G$1" pin="1"/>
-<wire x1="119.38" y1="-25.4" x2="119.38" y2="-30.48" width="0.1524" layer="91"/>
-<label x="119.38" y="-33.02" size="1.778" layer="95" rot="R90"/>
+<pinref part="U$2" gate="G$1" pin="VCC"/>
+<wire x1="-55.88" y1="-27.94" x2="-55.88" y2="-45.72" width="0.1524" layer="91"/>
+<wire x1="-55.88" y1="-45.72" x2="-71.12" y2="-45.72" width="0.1524" layer="91"/>
+<wire x1="-71.12" y1="-45.72" x2="-71.12" y2="43.18" width="0.1524" layer="91"/>
+<pinref part="U$4" gate="G$1" pin="5V"/>
+<wire x1="-71.12" y1="43.18" x2="-27.94" y2="43.18" width="0.1524" layer="91"/>
+<wire x1="-27.94" y1="43.18" x2="1.524" y2="43.18" width="0.1524" layer="91"/>
+<wire x1="-27.94" y1="43.18" x2="-27.94" y2="50.8" width="0.1524" layer="91"/>
+<junction x="-27.94" y="43.18"/>
+<label x="-27.94" y="50.8" size="1.778" layer="95"/>
 </segment>
 </net>
