File: Placa do Paraquedas - 1 skib/Esquema.brd (EAGLE design)
At the start: 160 x 100 mm, 14 parts, among them Q1 IRF540

Commit message: Update
Parts:
- removed S2: (no value), pinhead:1X01
Connections:
- removed net SINAL_SKIB2: S2.1
Changed lines of the file:
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@@
 <attribute name="VALUE" x="62.23" y="33.655" size="1.27" layer="27"/>
-</element>
-<element name="S2" library="pinhead" library_urn="urn:adsk.eagle:library:325" package="1X01" package3d_urn="urn:adsk.eagle:package:22485/2" value="" x="66.04" y="36.83" smashed="yes">
-<attribute name="NAME" x="64.6938" y="38.6588" size="1.27" layer="25" ratio="10"/>
-<attribute name="POPULARITY" value="64" x="66.04" y="36.83" size="1.778" layer="27" display="off"/>
-<attribute name="VALUE" x="64.77" y="33.655" size="1.27" layer="27"/>
 </element>
 </elements>
@@
 <wire x1="41.91" y1="38.1254" x2="41.91" y2="45.72" width="1" layer="1"/>
 </signal>
-<signal name="SINAL_SKIB2">
-<contactref element="S2" pad="1"/>
-</signal>
 </signals>
