File: Placa do Paraquedas - 1 skib/Esquema.sch (EAGLE design)
At the start: 14 parts, among them Q1 IRF540

Commit message: Update
Parts:
- removed S2: (no value), pinhead:PINHD-1X1
Connections:
- removed net SINAL_SKIB2: S2.1
Other:
- note added: "Entradas: - Bateria-1: Positivo da bateria de 3.7V - Bateria-2: Negativo da bateria de 3.7V - 3.3V: 3.3V do ESP32 - Parachute: Sinal de ativação do Paraquedas do ESP32 - Buzzer: Sinal do Buzzer do ESP32 Saídas: - Sinal_skib1: Sinal que identifica se o SKIB1 foi plugado OBS.: Quando: - Sinal_skib1: 0 - Parachute: 0 Significa que o skib não foi plugado. Quando: - Sinal_skib1: 0 - Parachute: 1 Signi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"
- note removed: "Entradas: - Bateria-1: Positivo da bateria de 3.7V - Bateria-2: Negativo da bateria de 3.7V - 3.3V: 3.3V do ESP32 - Parachute: Sinal de ativação do Paraquedas do ESP32 - Buzzer: Sinal do Buzzer do ESP32 Saídas: - Sinal_skib1: Sinal que identifica se o SKIB1 foi plugado - Sinal_skib2: Sinal que identifica se o SKIB2 foi plugado OBS.: Quando: - Sinal_skib1: 0 - Sinal_skib2: 0 - Parachute: 0 Signifi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"
Changed lines of the file:
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@@
 <part name="E3" library="pinhead" library_urn="urn:adsk.eagle:library:325" deviceset="PINHD-1X1" device="" package3d_urn="urn:adsk.eagle:package:22485/2"/>
 <part name="S1" library="pinhead" library_urn="urn:adsk.eagle:library:325" deviceset="PINHD-1X1" device="" package3d_urn="urn:adsk.eagle:package:22485/2"/>
-<part name="S2" library="pinhead" library_urn="urn:adsk.eagle:library:325" deviceset="PINHD-1X1" device="" package3d_urn="urn:adsk.eagle:package:22485/2"/>
 </parts>
 <sheets>
 <sheet>
 <plain>
-<text x="0" y="91.44" size="2.54" layer="91">Entradas:
+<text x="-10.16" y="93.98" size="2.54" layer="91">Entradas:
 - Bateria-1: Positivo da bateria de 3.7V
 - Bateria-2: Negativo da bateria de 3.7V
@@
 Saídas:
 - Sinal_skib1: Sinal que identifica se o SKIB1 foi plugado
-- Sinal_skib2: Sinal que identifica se o SKIB2 foi plugado
 OBS.:
 Quando:
 - Sinal_skib1: 0
-- Sinal_skib2: 0
 - Parachute: 0
-Significa que os skibs não foram plugados.
+Significa que o skib não foi plugado.
 Quando:
 - Sinal_skib1: 0
-- Sinal_skib2: 0
 - Parachute: 1
-Significa que os skibs haviam sido plugados, mas o sistema já os acionou.</text>
+Significa que o skib havia sido plugado, mas o sistema já o acionou.</text>
 </plain>
 <instances>
@@
 <attribute name="NAME" x="168.91" y="66.675" size="1.778" layer="95"/>
 <attribute name="VALUE" x="168.91" y="58.42" size="1.778" layer="96"/>
-</instance>
-<instance part="S2" gate="G$1" x="175.26" y="53.34" smashed="yes">
-<attribute name="NAME" x="168.91" y="56.515" size="1.778" layer="95"/>
-<attribute name="VALUE" x="168.91" y="48.26" size="1.778" layer="96"/>
 </instance>
 </instances>
@@
 </segment>
 </net>
-<net name="SINAL_SKIB2" class="0">
-<segment>
-<wire x1="142.24" y1="60.96" x2="162.56" y2="60.96" width="0.1524" layer="91"/>
-<label x="142.24" y="58.42" size="1.778" layer="95"/>
-<wire x1="162.56" y1="60.96" x2="162.56" y2="53.34" width="0.1524" layer="91"/>
-<pinref part="S2" gate="G$1" pin="1"/>
-<wire x1="162.56" y1="53.34" x2="172.72" y2="53.34" width="0.1524" layer="91"/>
-</segment>
-</net>
